Commit message: Fix simulation physics: invert right wheel commands, reduce friction, simplify control logic

File: src/amiga_sim/urdf/amiga_model_v1.urdf (robot description, URDF)
Before this commit: robot amiga_model, 34 links, 33 joints
Links:
- added link wheel_center, mass 0.001
Joints:
- added joint wheel_center_joint: type fixed, parent base_footprint, child wheel_center, origin xyz=0.593 0.399 0.429 rpy=0 0 0
